Commit message: cannot right place

File: models/cannon.urdf (robot description, URDF)
Before this commit: robot cannon, 3 links, 2 joints
Links:
- removed link cannonball
Joints:
- removed joint barrel_to_cannonball
- joint base_to_barrel: axis 0 1 0 -> (none); limit lower=-0.5 upper=1.5 effort=1000.0 velocity=0.5 -> (none); origin xyz=0 0 0.25 rpy=0 0 0 -> xyz=0 0 0.25 rpy=0 1.5707963267948966 0; type revolute -> fixed
